File: Schematic&PCB/KiCad/Regulus Focuser-V1.1/RegulusFocuser-V1.1.kicad_pcb (KiCad board)
At the start: 4 copper layers, 86.4 x 49.5 mm, 51 parts, among them J1 USB_A, J2 Display&Encoder, J3 Serial1, J4 R-Connect, J5 MotorPower, J6 MotorConnector, J7 5V-Ext, J8 LimiterSW, J9 ResetSW, U1 FT232RL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

Commit message: Code was adapted for the new INDI library v2.1.4, CMakeLists.txt optimised
Parts:
- turned R2 to 90 degrees
- turned R3 to 90 degrees
Connections:
- R2 pad 2: GND -> /3V3
- R3 pad 2: GND -> /3V3
Routing:
- net GND: track 19.1 -> 333.7 mm, vias 4 -> 2
- net /5V: track 269.9 -> 252.8 mm, vias 2 -> 0
- net Net-(J1-D-): track 36.3 -> 27.4 mm
- net /485RO: track 50.0 -> 45.6 mm
- net Net-(D3-A): track 16.5 -> 20.8 mm
- net Net-(J1-D+): track 37.2 -> 33.2 mm
- net Net-(D2-A): track 20.4 -> 16.6 mm
- net /SDA-2: track 26.3 -> 29.9 mm, vias 0 -> 1
- net /LimiterSwitch: track 58.2 -> 55.0 mm
- net /485DE: track 42.9 -> 39.9 mm
- net /3V3: track 121.1 -> 119.1 mm
- net /SCL-2: track 31.2 -> 32.8 mm, vias 0 -> 1
- net /L485DI: track 35.9 -> 34.4 mm
- net Net-(D1-K): track 22.6 -> 24.0 mm, vias 0 -> 2
- net Net-(J6-Pin_2): track 21.7 -> 22.9 mm
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- added copper zone on In2.Cu, net /3V3
- added copper zone on B.Cu, net /5V
- added copper zone on In1.Cu, net GND
- removed copper zone on B.Cu, net GND
