File: Schematic&PCB/KiCad/Regulus Focuser-V1.1/RegulusFocuser-V1.1.kicad_sch (KiCad schematic)
At the start: 47 parts, among them J1 USB_A, J2 Display&Encoder, J3 Serial1, J4 R-Connect, J5 MotorPower, J6 MotorConnector, J7 5V-Ext, J8 LimiterSW, J9 ResetSW, U1 FT232RL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

Commit message: Code was adapted for the new INDI library v2.1.4, CMakeLists.txt optimised
Connections:
- net 3V3: now also R2.2, R3.2
- net GND: no longer R2.2, R3.2

Commit message: Added backlash aid in firmware
Changed lines of the file:
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@@
 (kicad_sch
-	(version 20231120)
+	(version 20250114)
 	(generator "eeschema")
-	(generator_version "8.0")
+	(generator_version "9.0")
 	(paper "A4")
 	(title_block
@@
 	(label "3V3"
 		(at 200.66 114.3 0)
-		(fields_autoplaced yes)
 		(effects
 			(font
@@
 	(label "MODBUS+"
 		(at 180.34 143.51 0)
-		(fields_autoplaced yes)
 		(effects
 			(font
@@
 	(label "L485DE"
 		(at 120.65 95.25 180)
-		(fields_autoplaced yes)
 		(effects
 			(font
@@
 	(label "TX2"
 		(at 44.45 86.36 0)
-		(fields_autoplaced yes)
 		(effects
 			(font
@@
 	(label "EncDt"
 		(at 165.1 46.99 0)
-		(fields_autoplaced yes)
 		(effects
 			(font
@@
 	(label "M3"
 		(at 200.66 121.92 0)
-		(fields_autoplaced yes)
 		(effects
 			(font
@@
 	(label "3V3"
 		(at 245.11 129.54 0)
-		(fields_autoplaced yes)
 		(effects
 			(font
@@
 	(label "L485DE"
 		(at 165.1 52.07 0)
-		(fields_autoplaced yes)
 		(effects
 			(font
@@
 	(label "5V"
 		(at 176.53 160.02 0)
-		(fields_autoplaced yes)
 		(effects
 			(font
@@
 	(label "FLT"
 		(at 198.12 54.61 0)
-		(fields_autoplaced yes)
 		(effects
 			(font
@@
 	(label "L485RO"
 		(at 165.1 59.69 0)
-		(fields_autoplaced yes)
 		(effects
 			(font
@@
 	(label "M1"
 		(at 198.12 46.99 0)
-		(fields_autoplaced yes)
 		(effects
 			(font
@@
 	(label "Enable"
 		(at 198.12 41.91 0)
-		(fields_autoplaced yes)
 		(effects
 			(font
@@
 	(label "485DI"
 		(at 88.9 87.63 180)
-		(fields_autoplaced yes)
 		(effects
 			(font
@@
 	(label "485RO"
 		(at 88.9 85.09 180)
-		(fields_autoplaced yes)
 		(effects
 			(font
@@
 	(label "SCL-2"
 		(at 40.64 50.8 0)
-		(fields_autoplaced yes)
 		(effects
 			(font
@@
 	(label "M1"
 		(at 200.66 116.84 0)
-		(fields_autoplaced yes)
 		(effects
 			(font
@@
 	(label "SCL-2"
 		(at 198.12 57.15 0)
-		(fields_autoplaced yes)
 		(effects
 			(font
@@
 	(label "5V"
 		(at 38.1 175.26 0)
-		(fields_autoplaced yes)
 		(effects
 			(font
@@
 	(label "L485DI"
 		(at 165.1 57.15 0)
-		(fields_autoplaced yes)
 		(effects
 			(font
@@
 	(label "STDBY"
 		(at 198.12 44.45 0)
-		(fields_autoplaced yes)
 		(effects
 			(font
@@
 	(label "EncClk"
 		(at 44.45 58.42 0)
-		(fields_autoplaced yes)
 		(effects
 			(font
@@
 	(label "485DE"
 		(at 137.16 41.91 0)
-		(fields_autoplaced yes)
 		(effects
 			(font
@@
 	(label "Step"
 		(at 200.66 129.54 0)
-		(fields_autoplaced yes)
 		(effects
 			(font
@@
 	(label "3V3"
 		(at 233.68 63.5 0)
-		(fields_autoplaced yes)
 		(effects
 			(font
@@
 	(label "M3"
 		(at 198.12 52.07 0)
-		(fields_autoplaced yes)
 		(effects
 			(font
@@
 	(label "RX2"
 		(at 165.1 41.91 0)
-		(fields_autoplaced yes)
 		(effects
 			(font
@@
 	(label "RX2"
 		(at 44.45 88.9 0)
-		(fields_autoplaced yes)
 		(effects
 			(font
@@
 	(label "FLT"
 		(at 200.66 124.46 0)
-		(fields_autoplaced yes)
 		(effects
 			(font
@@
 	(label "L485RO"
 		(at 120.65 85.09 180)
-		(fields_autoplaced yes)
 		(effects
 			(font
@@
 	(label "L485DI"
 		(at 113.03 87.63 0)
-		(fields_autoplaced yes)
 		(effects
 			(font
@@
 	(label "SDA-2"
 		(at 198.12 59.69 0)
-		(fields_autoplaced yes)
 		(effects
 			(font
@@
 	(label "Enable"
 		(at 200.66 109.22 0)
-		(fields_autoplaced yes)
 		(effects
 			(font
@@
 	(label "3V3"
 		(at 222.25 41.91 0)
-		(fields_autoplaced yes)
 		(effects
 			(font
@@
 	(label "STDBY"
 		(at 200.66 127 0)
-		(fields_autoplaced yes)
 		(effects
 			(font
@@
 	(label "485DE"
 		(at 88.9 95.25 180)
-		(fields_autoplaced yes)
 		(effects
 			(font
@@
 	(label "485RO"
 		(at 137.16 46.99 0)
-		(fields_autoplaced yes)
 		(effects
 			(font
@@
 	(label "EncSw"
 		(at 44.45 63.5 0)
-		(fields_autoplaced yes)
 		(effects
 			(font
@@
 	(label "5V"
 		(at 165.1 21.59 0)
-		(fields_autoplaced yes)
 		(effects
 			(font
@@
 	(label "LimiterSwitch"
 		(at 198.12 62.23 0)
-		(fields_autoplaced yes)
 		(effects
 			(font
@@
 	(label "5V"
 		(at 62.23 46.99 0)
-		(fields_autoplaced yes)
 		(effects
 			(font
@@
 	(label "EncDt"
 		(at 44.45 60.96 0)
-		(fields_autoplaced yes)
 		(effects
 			(font
@@
 	(label "3V3"
 		(at 116.84 90.17 180)
-		(fields_autoplaced yes)
 		(effects
 			(font
@@
 	(label "Reset"
 		(at 198.12 74.93 0)
-		(fields_autoplaced yes)
 		(effects
 			(font
@@
 	(label "5V"
 		(at 129.54 189.23 0)
-		(fields_autoplaced yes)
 		(effects
 			(font
@@
 	(label "Buzzer"
 		(at 165.1 34.29 0)
-		(fields_autoplaced yes)
 		(effects
 			(font
@@
 	(label "TX2"
 		(at 165.1 39.37 0)
-		(fields_autoplaced yes)
 		(effects
 			(font
@@
 	(label "3V3"
 		(at 198.12 19.05 0)
-		(fields_autoplaced yes)
 		(effects
 			(font
@@
 	(label "LimiterSwitch"
 		(at 222.25 38.1 0)
-		(fields_autoplaced yes)
 		(effects
 			(font
@@
 	(label "Reset"
 		(at 233.68 58.42 0)
-		(fields_autoplaced yes)
 		(effects
 			(font
@@
 	(label "EncSw"
 		(at 165.1 44.45 0)
-		(fields_autoplaced yes)
 		(effects
 			(font
@@
 	(label "5V"
 		(at 246.38 25.4 0)
-		(fields_autoplaced yes)
 		(effects
 			(font
@@
 	(label "MODBUS-"
 		(at 62.23 44.45 0)
-		(fields_autoplaced yes)
 		(effects
 			(font
@@
 	(label "Buzzer"
 		(at 44.45 99.06 0)
-		(fields_autoplaced yes)
 		(effects
 			(font
@@
 	(label "5V"
 		(at 33.02 124.46 0)
-		(fields_autoplaced yes)
 		(effects
 			(font
@@
 	(label "5V"
 		(at 86.36 90.17 180)
-		(fields_autoplaced yes)
 		(effects
 			(font
@@
 	(label "Direction"
 		(at 200.66 132.08 0)
-		(fields_autoplaced yes)
 		(effects
 			(font
@@
 	(label "SDA-2"
 		(at 40.64 48.26 0)
-		(fields_autoplaced yes)
 		(effects
 			(font
@@
 	(label "EncClk"
 		(at 165.1 49.53 0)
-		(fields_autoplaced yes)
 		(effects
 			(font
@@
 	(label "485DI"
 		(at 137.16 39.37 0)
-		(fields_autoplaced yes)
 		(effects
 			(font
@@
 	(label "M2"
 		(at 200.66 119.38 0)
-		(fields_autoplaced yes)
 		(effects
 			(font
@@
 	(label "3V3"
 		(at 40.64 53.34 0)
-		(fields_autoplaced yes)
 		(effects
 			(font
@@
 	(label "MODBUS+"
 		(at 62.23 41.91 0)
-		(fields_autoplaced yes)
 		(effects
 			(font
@@
 	(label "MODBUS-"
 		(at 180.34 140.97 0)
-		(fields_autoplaced yes)
 		(effects
 			(font
@@
 	(label "M2"
 		(at 198.12 49.53 0)
-		(fields_autoplaced yes)
 		(effects
 			(font
@@
 	(label "Direction"
 		(at 198.12 39.37 0)
-		(fields_autoplaced yes)
 		(effects
 			(font
@@
 	(label "Step"
 		(at 198.12 36.83 0)
-		(fields_autoplaced yes)
 		(effects
 			(font
@@
 	(label "3V3"
 		(at 45.72 27.94 0)
-		(fields_autoplaced yes)
 		(effects
 			(font
@@
 		)
 	)
+	(embedded_fonts no)
 )
